Commit message: amp_kart_description: added new joints
Added two new joints to the racecar.xacro file. Velodyne and zed camera
center joints.

File: src/amp_kart_description/urdf/racecar.xacro (robot description, xacro)
@@ -154,5 +154,5 @@
   <xacro:VLP-16
     parent="chassis"
-    name="laser"
+    name="velodyne"
     topic="/velodyne_points"
     hz="10"
@@ -162,30 +162,4 @@
   <origin xyz="0.265 0.0 0.075" rpy="0 0 0" />
   </xacro:VLP-16>
-  <!-- Add Hokuyo laser scanner -->
-<!--
-  <link name="laser">
-    <inertial>
-      <xacro:hokuyo_inertial_params />
-    </inertial>
-    <collision>
-      <origin xyz="0 0 0" rpy="0 0 0" />
-      <geometry>
-        <box size="0.1 0.1 0.1" />
-      </geometry>
-    </collision>
-    <visual>
-      <origin xyz="0 0 0" rpy="0 0 0" />
-      <geometry>
-        <!<mesh filename="package://amp_cart_description/meshes/hokuyo.dae" />
-        <material name="grey" />
-      </geometry>
-    </visual>
-  </link>
-  <joint name="hokuyo_joint" type="fixed">
-    <origin xyz="0.265 0.0 0.075" rpy="0 0 0" />
-    <parent link="chassis" />
-    <child link="laser" />
-    <axis xyz="0 0 1" />
-  </joint> -->
   <!-- zed camera -->
   <link name="zed_camera_link">
@@ -234,4 +208,11 @@
     </inertial>
   </link>
+  <link name="zed_camera_center">
+    <inertial>
+      <mass value="1e-5" />
+      <origin xyz="0 0 0" rpy="0 0 0" />
+      <inertia ixx="1e-6" ixy="0" ixz="0" iyy="1e-6" iyz="0" izz="1e-6" />
+    </inertial>
+  </link>
   <joint name="zed_camera_left_joint" type="fixed">
     <origin xyz="0 0.06 0" rpy="0 0 0" />
@@ -246,4 +227,10 @@
     <axis xyz="0 0 1" />
   </joint>
+  <joint name="zed_camera_center_joint" type="fixed">
+    <origin xyz="0 0 0" rpy="0 0 0" />
+    <parent link="zed_camera_link" />
+    <child link="zed_camera_center" />
+    <axis xyz="0 0 1" />
+  </joint>
   <!-- Add the remaining xacros -->
   <xacro:include filename="$(find amp_kart_description)/urdf/racecar.gazebo" />

Commit message: amp_kart_description: changed racecar.xacro
Changed the sensor positionings to
 be more accurate to the irl kart.

File: src/amp_kart_description/urdf/racecar.xacro (robot description, xacro)
@@ -23,5 +23,5 @@
   <xacro:property name="chassisInertia_yoff" value="0" />
   <xacro:property name="chassisInertia_zoff" value="0" />
-  <xacro:property name="baseLink_xoff" value="-0.25" />
+  <xacro:property name="baseLink_xoff" value="0" />
   <xacro:property name="baseLink_yoff" value="0" />
   <xacro:property name="baseLink_zoff" value="0.05" />
@@ -44,11 +44,11 @@
   <xacro:property name="rfront_yoff" value="0" />
   <xacro:property name="rfront_zoff" value="0" />
-  <xacro:property name="lidar_xoff" value="0.25" />
-  <xacro:property name="lidar_zoff" value="0.4064" />
+  <xacro:property name="lidar_xoff" value="1.2192" />
+  <xacro:property name="lidar_zoff" value="0.4826" />
   <xacro:property name="zed_width" value="0.175" />
   <xacro:property name="zed_length" value="0.033" />
   <xacro:property name="zed_height" value="0.03" />
-  <xacro:property name="zed_xoff" value="0" />
-  <xacro:property name="zed_zoff" value="0.3048" />
+  <xacro:property name="zed_xoff" value="1.27" />
+  <xacro:property name="zed_zoff" value="0.4064" />
   <xacro:property name="zed_mass" value="0.02" />
   <!-- Add chassis and it's inertia link -->
@@ -252,5 +252,5 @@
   </link>
   <joint name="zed_camera_joint" type="continuous">
-    <origin xyz="0.390 0 0.04" rpy="0 0 0" />
+    <origin xyz="0 0 0" rpy="0 0 0" />
     <parent link="chassis" />
     <child link="zed_camera_link" />

Commit message: amp_kart_description: modify and simplify urdf
Removed unnecessary links and joints for zed, as well as modified
dimensions slightly.

File: src/amp_kart_description/urdf/racecar.xacro (robot description, xacro)
@@ -45,10 +45,10 @@
   <xacro:property name="rfront_zoff" value="0" />
   <xacro:property name="lidar_xoff" value="1.2192" />
-  <xacro:property name="lidar_zoff" value="0.4826" />
+  <xacro:property name="lidar_zoff" value="0.508" />
   <xacro:property name="zed_width" value="0.175" />
   <xacro:property name="zed_length" value="0.033" />
   <xacro:property name="zed_height" value="0.03" />
   <xacro:property name="zed_xoff" value="1.27" />
-  <xacro:property name="zed_zoff" value="0.4064" />
+  <xacro:property name="zed_zoff" value="0.381" />
   <xacro:property name="zed_mass" value="0.02" />
   <!-- Add chassis and it's inertia link -->
@@ -234,9 +234,9 @@
     <inertial>
       <mass value="1e-5" />
-      <origin xyz="${zed_xoff} 0 ${zed_zoff}" rpy="0 0 0" />
+      <origin xyz="0 0 0" rpy="0 0 0" />
       <inertia ixx="1e-6" ixy="0" ixz="0" iyy="1e-6" iyz="0" izz="1e-6" />
     </inertial>
     <collision>
-      <origin xyz="${zed_xoff} 0 ${zed_zoff}" rpy="0 0 0" />
+      <origin xyz="0 0 0" rpy="0 0 0" />
       <geometry>
         <box size="${zed_length} ${zed_width} ${zed_height}" />
@@ -244,5 +244,5 @@
     </collision>
     <visual>
-      <origin xyz="${zed_xoff} 0 ${zed_zoff}" rpy="0 0 0" />
+      <origin xyz="0 0 0" rpy="0 0 0" />
       <geometry>
         <box size="${zed_length} ${zed_width} ${zed_height}" />
@@ -253,5 +253,5 @@
   <joint name="zed_camera_joint" type="continuous">
     <origin xyz="0 0 0" rpy="0 0 0" />
-    <parent link="chassis" />
+    <parent link="zed_camera_center" />
     <child link="zed_camera_link" />
     <axis xyz="0 0 1" />
@@ -259,43 +259,14 @@
   </joint>
   <!-- zed camera lenses -->
-  <!-- It seems these have to have a non-zero mass to have a camera attached? -->
-  <link
-    name="camera_link"
-  ><!-- this needs to match the name in zed_wrapper/zed_tf.launch -->
+  <link name="zed_camera_center">
     <inertial>
       <mass value="1e-5" />
-      <origin xyz="${zed_xoff} 0 ${zed_zoff}" rpy="0 0 0" />
+      <origin xyz="0 0 0" rpy="0 0 0" />
       <inertia ixx="1e-6" ixy="0" ixz="0" iyy="1e-6" iyz="0" izz="1e-6" />
     </inertial>
   </link>
-  <link name="zed_camera_right_link">
-    <inertial>
-      <mass value="1e-5" />
-      <origin xyz="${zed_xoff} 0 ${zed_zoff}" rpy="0 0 0" />
-      <inertia ixx="1e-6" ixy="0" ixz="0" iyy="1e-6" iyz="0" izz="1e-6" />
-    </inertial>
-  </link>
-  <link name="zed_camera_center">
-    <inertial>
-      <mass value="1e-5" />
-      <origin xyz="${zed_xoff} 0 ${zed_zoff}" rpy="0 0 0" />
-      <inertia ixx="1e-6" ixy="0" ixz="0" iyy="1e-6" iyz="0" izz="1e-6" />
-    </inertial>
-  </link>
-  <joint name="zed_camera_left_joint" type="fixed">
-    <origin xyz="${zed_xoff} 0.06 ${zed_zoff}" rpy="0 0 0" />
-    <parent link="zed_camera_link" />
-    <child link="camera_link" />
-    <axis xyz="0 0 1" />
-  </joint>
-  <joint name="zed_camera_right_joint" type="fixed">
-    <origin xyz="${zed_xoff} -0.06 ${zed_zoff}" rpy="0 0 0" />
-    <parent link="zed_camera_link" />
-    <child link="zed_camera_right_link" />
-    <axis xyz="0 0 1" />
-  </joint>
   <joint name="zed_camera_center_joint" type="fixed">
     <origin xyz="${zed_xoff} 0 ${zed_zoff}" rpy="0 0 0" />
-    <parent link="zed_camera_link" />
+    <parent link="base_link" />
     <child link="zed_camera_center" />
     <axis xyz="0 0 1" />

Commit message: amp_kart_bringup: fix zed urdf issues
needed to remove zed camera from urdf since they were overwriting each
other. added zed launch as well.

File: src/amp_kart_description/urdf/racecar.xacro (robot description, xacro)
@@ -221,5 +221,5 @@
   />
   <xacro:VLP-16
-    parent="chassis"
+    parent="base_link"
     name="velodyne"
     topic="/velodyne_points"
@@ -231,5 +231,5 @@
   </xacro:VLP-16>
   <!-- zed camera -->
-  <link name="zed_camera_link">
+  <!-- <link name="zed_camera_link">
     <inertial>
       <mass value="1e-5" />
@@ -256,7 +256,5 @@
     <child link="zed_camera_link" />
     <axis xyz="0 0 1" />
-    <!-- <limit lower="0.0" upper="0.0" effort="0.0" velocity="0.0" /> -->
-  </joint>
-  <!-- zed camera lenses -->
+  </joint>
   <link name="zed_camera_center">
     <inertial>
@@ -271,5 +269,5 @@
     <child link="zed_camera_center" />
     <axis xyz="0 0 1" />
-  </joint>
+  </joint> -->
   <!-- Add the remaining xacros -->
   <xacro:include filename="$(find amp_kart_description)/urdf/racecar.gazebo" />

Commit message: clean up unnecessary files
removed unnecessary files and cleaned `racecar.xacro`.

File: src/amp_kart_description/urdf/racecar.xacro (robot description, xacro)
@@ -46,10 +46,4 @@
   <xacro:property name="lidar_xoff" value="1.2192" />
   <xacro:property name="lidar_zoff" value="0.508" />
-  <xacro:property name="zed_width" value="0.175" />
-  <xacro:property name="zed_length" value="0.033" />
-  <xacro:property name="zed_height" value="0.03" />
-  <xacro:property name="zed_xoff" value="1.27" />
-  <xacro:property name="zed_zoff" value="0.381" />
-  <xacro:property name="zed_mass" value="0.02" />
   <!-- Add chassis and it's inertia link -->
   <link name="base_link" />
@@ -216,6 +210,6 @@
   </joint>
   <xacro:wheel_transmission name="right_front_wheel" />
-  <!-- New Lidar Sensor-->
-   <xacro:include
+  <!-- VLP-16 -->
+  <xacro:include
     filename="$(find velodyne_description)/urdf/VLP-16.urdf.xacro"
   />
@@ -230,44 +224,4 @@
   <origin xyz="${lidar_xoff} 0 ${lidar_zoff}" rpy="0 0 0" />
   </xacro:VLP-16>
-  <!-- zed camera -->
-  <!-- <link name="zed_camera_link">
-    <inertial>
-      <mass value="1e-5" />
-      <origin xyz="0 0 0" rpy="0 0 0" />
-      <inertia ixx="1e-6" ixy="0" ixz="0" iyy="1e-6" iyz="0" izz="1e-6" />
-    </inertial>
-    <collision>
-      <origin xyz="0 0 0" rpy="0 0 0" />
-      <geometry>
-        <box size="${zed_length} ${zed_width} ${zed_height}" />
-      </geometry>
-    </collision>
-    <visual>
-      <origin xyz="0 0 0" rpy="0 0 0" />
-      <geometry>
-        <box size="${zed_length} ${zed_width} ${zed_height}" />
-      </geometry>
-      <material name="red" />
-    </visual>
-  </link>
-  <joint name="zed_camera_joint" type="continuous">
-    <origin xyz="0 0 0" rpy="0 0 0" />
-    <parent link="zed_camera_center" />
-    <child link="zed_camera_link" />
-    <axis xyz="0 0 1" />
-  </joint>
-  <link name="zed_camera_center">
-    <inertial>
-      <mass value="1e-5" />
-      <origin xyz="0 0 0" rpy="0 0 0" />
-      <inertia ixx="1e-6" ixy="0" ixz="0" iyy="1e-6" iyz="0" izz="1e-6" />
-    </inertial>
-  </link>
-  <joint name="zed_camera_center_joint" type="fixed">
-    <origin xyz="${zed_xoff} 0 ${zed_zoff}" rpy="0 0 0" />
-    <parent link="base_link" />
-    <child link="zed_camera_center" />
-    <axis xyz="0 0 1" />
-  </joint> -->
   <!-- Add the remaining xacros -->
   <xacro:include filename="$(find amp_kart_description)/urdf/racecar.gazebo" />

Commit message: Added adaptive clustering for lidars. WARNING: This branch has a problem with the URDF

File: src/amp_kart_description/urdf/racecar.xacro (robot description, xacro)
@@ -44,4 +44,6 @@
   <xacro:property name="rfront_yoff" value="0" />
   <xacro:property name="rfront_zoff" value="0" />
+  <!--xacro:property name="lidar_xoff" value="0.7239" />
+  <xacro:property name="lidar_zoff" value="0.38" /-->
   <xacro:property name="lidar_xoff" value="1.2192" />
   <xacro:property name="lidar_zoff" value="0.508" />
